Commit message: Under-actuated RH8D Gazebo simulation

File: v2_rh8d_ws/src/rh8d_control/description/rh8dL_ros2_control.xacro (robot description, xacro)
@@ -6,5 +6,5 @@
         <plugin>gz_ros2_control/GazeboSimSystem</plugin>
       </hardware>
-      <!-- Wrist / palm chain -->
+      <!-- Wrist / palm chain each joint has a seperate motor-->
       <joint name="forearm:1--base:1">
         <command_interface name="position"/>
@@ -22,5 +22,6 @@
         <state_interface name="velocity"/>
       </joint>
-      <!-- Thumb -->
+      <!-- Thumb share TWO motors -->
+      <!-- Actuated joint -->
       <joint name="Thumb_axis--palmL:1">
         <command_interface name="position"/>
@@ -29,81 +30,114 @@
       </joint>
       <joint name="Thumb_Methacarpal--Thumb_axis">
-        <command_interface name="position"/>
+        <command_interface name="effort"/>
         <state_interface name="position"/>
         <state_interface name="velocity"/>
+        <state_interface name="effort"/>
       </joint>
+      <!-- Thumb passive joints -->
       <joint name="Thumb_Proximal--Thumb_Methacarpal">
-        <command_interface name="position"/>
+        <param name="mimic">Thumb_Methacarpal--Thumb_axis</param>
+        <param name="multiplier">0.9</param>
         <state_interface name="position"/>
         <state_interface name="velocity"/>
+        <state_interface name="effort"/>
       </joint>
       <joint name="Thumb_Distal--Thumb_Proximal">
-        <command_interface name="position"/>
+        <param name="mimic">Thumb_Proximal--Thumb_Methacarpal</param>
+        <param name="multiplier">0.9</param>
         <state_interface name="position"/>
         <state_interface name="velocity"/>
+        <state_interface name="effort"/>
       </joint>
-      <!-- Index -->
+      <!-- Index share ONE motor -->
+      <!-- Actuated joint -->
       <joint name="Index_Proximal--palmL:1">
-        <command_interface name="position"/>
+        <command_interface name="effort"/>
         <state_interface name="position"/>
         <state_interface name="velocity"/>
+        <state_interface name="effort"/>
       </joint>
+      <!-- Index passive joints -->
       <joint name="Index_Middle--Index_Proximal">
-        <command_interface name="position"/>
+        <param name="mimic">Index_Proximal--palmL:1</param>
+        <param name="multiplier">0.9</param>
         <state_interface name="position"/>
         <state_interface name="velocity"/>
+        <state_interface name="effort"/>
       </joint>
       <joint name="Index_Distal--Index_Middle">
-        <command_interface name="position"/>
+        <param name="mimic">Index_Middle--Index_Proximal</param>
+        <param name="multiplier">0.9</param>
         <state_interface name="position"/>
         <state_interface name="velocity"/>
+        <state_interface name="effort"/>
       </joint>
-      <!-- Middle -->
+      <!-- Middle share ONE motor -->
+      <!-- Actuated joint -->
       <joint name="Middle_Proximal--palmL:1">
-        <command_interface name="position"/>
+        <command_interface name="effort"/>
         <state_interface name="position"/>
         <state_interface name="velocity"/>
+        <state_interface name="effort"/>
       </joint>
+      <!-- Middle passive joints -->
       <joint name="Middle_Middle--Middle_Proximal">
-        <command_interface name="position"/>
+        <param name="mimic">Middle_Proximal--palmL:1</param>
+        <param name="multiplier">0.9</param>
         <state_interface name="position"/>
         <state_interface name="velocity"/>
+        <state_interface name="effort"/>
       </joint>
       <joint name="Middle_Distal--Middle_Middle">
-        <command_interface name="position"/>
+        <param name="mimic">Middle_Middle--Middle_Proximal</param>
+        <param name="multiplier">0.9</param>
         <state_interface name="position"/>
         <state_interface name="velocity"/>
+        <state_interface name="effort"/>
       </joint>
-      <!-- Ring -->
+      <!-- Ring + Small share ONE motor -->
+      <!-- Actuated joint -->
       <joint name="Ring_Proximal--palmL:1">
-        <command_interface name="position"/>
+        <command_interface name="effort"/>
         <state_interface name="position"/>
         <state_interface name="velocity"/>
+        <state_interface name="effort"/>
       </joint>
+      <!-- Ring passive joints -->
       <joint name="Ring_Middle--Ring_Proximal">
-        <command_interface name="position"/>
+        <param name="mimic">Ring_Proximal--palmL:1</param>
+        <param name="multiplier">0.9</param>
         <state_interface name="position"/>
         <state_interface name="velocity"/>
+        <state_interface name="effort"/>
       </joint>
       <joint name="Ring_Distal--Ring_Middle">
-        <command_interface name="position"/>
+        <param name="mimic">Ring_Middle--Ring_Proximal</param>
+        <param name="multiplier">0.9</param>
         <state_interface name="position"/>
         <state_interface name="velocity"/>
+        <state_interface name="effort"/>
       </joint>
-      <!-- Small -->
+      <!-- Small passive joints -->
       <joint name="Small_Proximal--palmL:1">
-        <command_interface name="position"/>
-        <state_interface name="position"/>
-        <state_interface name="velocity"/>
+          <param name="mimic">Ring_Proximal--palmL:1</param>
+          <param name="multiplier">1.0</param>
+          <state_interface name="position"/>
+          <state_interface name="velocity"/>
+          <state_interface name="effort"/>
       </joint>
       <joint name="Small_Middle--Small_Proximal">
-        <command_interface name="position"/>
-        <state_interface name="position"/>
-        <state_interface name="velocity"/>
+          <param name="mimic">Small_Proximal--palmL:1</param>
+          <param name="multiplier">0.9</param>
+          <state_interface name="position"/>
+          <state_interface name="velocity"/>
+          <state_interface name="effort"/>
       </joint>
       <joint name="Small_Distal--Small_Middle">
-        <command_interface name="position"/>
-        <state_interface name="position"/>
-        <state_interface name="velocity"/>
+          <param name="mimic">Small_Middle--Small_Proximal</param>
+          <param name="multiplier">0.9</param>
+          <state_interface name="position"/>
+          <state_interface name="velocity"/>
+          <state_interface name="effort"/>
       </joint>
     </ros2_control>

File: v2_rh8d_ws/src/rh8d_description/gazebo/rh8dL_gazebo.xacro (robot description, xacro)
@@ -1,4 +1,6 @@
 <?xml version="1.0"?>
 <robot xmlns:xacro="http://www.ros.org/wiki/xacro">
+    <xacro:arg name="robot_controllers" default=""/>
+    <xacro:property name="robot_controllers" value="$(arg robot_controllers)"/>
     <!-- color definition -->
     <xacro:property name="silver" value="0.74902 0.74902 0.74902 1.0"/>
@@ -49,43 +51,43 @@
     <!-- PalmL:1 Link -->
     <xacro:gz_material link="palmL:1"/>
-    <xacro:gz_contact link="palmL:1" mu="1.2" kp="5e4" kd="80"/>
+    <xacro:gz_contact link="palmL:1" mu="1.5" kp="5e4" kd="80"/>
     <!-- Thumb Axis Link -->
     <xacro:gz_material link="Thumb_axis"/>
-    <xacro:gz_contact link="Thumb_axis" mu="1.2" kp="5e4" kd="80"/>
+    <xacro:gz_contact link="Thumb_axis" mu="1.5" kp="5e3" kd="30"/>
     <!-- Thumb Links -->
     <xacro:gz_material link="Thumb_Proximal"/>
-    <xacro:gz_contact link="Thumb_Proximal" mu="1.2" kp="5e4" kd="80"/>
+    <xacro:gz_contact link="Thumb_Proximal" mu="2.0" kp="5e3" kd="30" selfCollide="false"/>
     <xacro:gz_material link="Thumb_Methacarpal"/>
-    <xacro:gz_contact link="Thumb_Methacarpal" mu="1.2" kp="5e4" kd="80"/>
+    <xacro:gz_contact link="Thumb_Methacarpal" mu="2.0" kp="5e3" kd="30" selfCollide="false"/>
     <xacro:gz_material link="Thumb_Distal"/>
-    <xacro:gz_contact link="Thumb_Distal" mu="1.2" kp="5e4" kd="80"/>
+    <xacro:gz_contact link="Thumb_Distal" mu="2.0" kp="5e3" kd="30" selfCollide="false"/>
     <!-- Index Links -->
     <xacro:gz_material link="Index_Proximal"/>
-    <xacro:gz_contact link="Index_Proximal" mu="1.2" kp="5e4" kd="80"/>
+    <xacro:gz_contact link="Index_Proximal" mu="2.0" kp="5e3" kd="30" selfCollide="false"/>
     <xacro:gz_material link="Index_Middle"/>
-    <xacro:gz_contact link="Index_Middle" mu="1.2" kp="5e4" kd="80"/>
+    <xacro:gz_contact link="Index_Middle" mu="2.0" kp="5e3" kd="30" selfCollide="false"/>
     <xacro:gz_material link="Index_Distal"/>
-    <xacro:gz_contact link="Index_Distal" mu="1.2" kp="5e4" kd="80"/>
+    <xacro:gz_contact link="Index_Distal" mu="2.0" kp="5e3" kd="30" selfCollide="false"/>
     <!-- Middle Links -->
     <xacro:gz_material link="Middle_Proximal"/>
-    <xacro:gz_contact link="Middle_Proximal" mu="1.2" kp="5e4" kd="80"/>
+    <xacro:gz_contact link="Middle_Proximal" mu="2.0" kp="5e3" kd="30" selfCollide="false"/>
     <xacro:gz_material link="Middle_Middle"/>
-    <xacro:gz_contact link="Middle_Middle" mu="1.2" kp="5e4" kd="80"/>
+    <xacro:gz_contact link="Middle_Middle" mu="2.0" kp="5e3" kd="30" selfCollide="false"/>
     <xacro:gz_material link="Middle_Distal"/>
-    <xacro:gz_contact link="Middle_Distal" mu="1.2" kp="5e4" kd="80"/>
+    <xacro:gz_contact link="Middle_Distal" mu="2.0" kp="5e3" kd="30" selfCollide="false"/>
     <!-- Ring Links -->
     <xacro:gz_material link="Ring_Proximal"/>
-    <xacro:gz_contact link="Ring_Proximal" mu="1.2" kp="5e4" kd="80"/>
+    <xacro:gz_contact link="Ring_Proximal" mu="2.0" kp="5e3" kd="30" selfCollide="false"/>
     <xacro:gz_material link="Ring_Middle"/>
-    <xacro:gz_contact link="Ring_Middle" mu="1.2" kp="5e4" kd="80"/>
+    <xacro:gz_contact link="Ring_Middle" mu="2.0" kp="5e3" kd="30" selfCollide="false"/>
     <xacro:gz_material link="Ring_Distal"/>
-    <xacro:gz_contact link="Ring_Distal" mu="1.2" kp="5e4" kd="80"/>
+    <xacro:gz_contact link="Ring_Distal" mu="2.0" kp="5e3" kd="30" selfCollide="false"/>
     <!-- Small Links -->
     <xacro:gz_material link="Small_Proximal"/>
-    <xacro:gz_contact link="Small_Proximal" mu="1.2" kp="5e4" kd="80"/>
+    <xacro:gz_contact link="Small_Proximal" mu="2.0" kp="5e3" kd="30" selfCollide="false"/>
     <xacro:gz_material link="Small_Middle"/>
-    <xacro:gz_contact link="Small_Middle" mu="1.2" kp="5e4" kd="80"/>
+    <xacro:gz_contact link="Small_Middle" mu="2.0" kp="5e3" kd="30" selfCollide="false"/>
     <xacro:gz_material link="Small_Distal"/>
-    <xacro:gz_contact link="Small_Distal" mu="1.2" kp="5e4" kd="80"/>
+    <xacro:gz_contact link="Small_Distal" mu="2.0" kp="5e3" kd="30" selfCollide="false"/>
     <!-- Gazebo ROS2 Control Plugin -->
     <gazebo>
@@ -93,5 +95,5 @@
             <robot_param>robot_description</robot_param>
             <robot_param_node>robot_state_publisher</robot_param_node>
-        <parameters>$(find rh8d_control)/config/rh8dL_controllers.yaml</parameters>
+            <parameters>${robot_controllers}</parameters>
         </plugin>
     </gazebo>

File: v2_rh8d_ws/src/rh8d_description/urdf/rh8dL_base_forearm.xacro (robot description, xacro)
@@ -1,11 +1,14 @@
 <?xml version="1.0"?>
 <robot xmlns:xacro="http://www.ros.org/wiki/xacro">
-  <!-- Base link -->
-  <link name="base_link" />
-  <!-- Fixed joint: base_link -> base:1 -->
-  <joint name="base:1--base_link" type="fixed">
-    <parent link="base_link"/>
+  <!-- World -->
+  <link name="world" />
+  <!-- Fixed joint: world -> base:1 -->
+  <joint name="base:1--world" type="fixed">
+    <parent link="world"/>
     <child link="base:1"/>
-    <origin xyz="0 0 0" rpy="0 0 0"/>
+    <!-- For picking up Coke (side pick) -->
+    <!-- <origin xyz="0.35 0.6 1.047" rpy="0 -1.57079632679 3.14159265359"/>   -->
+    <!-- For picking up Ball (top pick)-->
+    <origin xyz="0.58 -0.13 1.045" rpy="-1.57079632679 0 0"/>
   </joint>
   <!-- Base:1 link -->
@@ -61,6 +64,6 @@
     <parent link="base:1"/>
     <child link="forearm:1"/>
-    <dynamics damping="0.1"/>
-    <limit effort="0.5" lower="-1.57079632679" upper="1.57079632679" velocity="1.0"/>
+    <dynamics damping="0.05" friction="0.005"/>
+    <limit effort="2.5" lower="-1.57079632679" upper="1.57079632679" velocity="5.0"/>
   </joint>
 </robot>

File: v2_rh8d_ws/src/rh8d_description/urdf/rh8dL_index.xacro (robot description, xacro)
@@ -26,10 +26,10 @@
     <!--Joint: palmL:1 -> Index_Proximal -->
     <joint name="Index_Proximal--palmL:1" type="revolute">
-    <origin xyz="0.015314 -0.080697 0.00509984" rpy="-1.76215945719 -0.155855069444 0.117563149369"/>
-    <axis xyz="-1.0 0.0 0.0"/>
-    <parent link="palmL:1"/>
-    <child link="Index_Proximal"/>
-    <dynamics damping="0.1"/>
-    <limit effort="0.5" lower="0" upper="1.57079632679" velocity="1.0"/>
+        <origin xyz="0.015314 -0.080697 0.00509984" rpy="-1.76215945719 -0.155855069444 0.117563149369"/>
+        <axis xyz="-1.0 0.0 0.0"/>
+        <parent link="palmL:1"/>
+        <child link="Index_Proximal"/>
+        <dynamics damping="0.05" friction="0.005"/>
+        <limit effort="2.5" lower="0" upper="1.57079632679" velocity="5.0"/>
     </joint>
     <!-- Index Middle -->
@@ -58,10 +58,13 @@
     <!--Joint: Index_Proximal -> Index_Middle -->
     <joint name="Index_Middle--Index_Proximal" type="revolute">
-    <origin xyz="6.2440782901e-05 0 -0.025875292969" rpy="0 0 0"/>
-    <axis xyz="-1.0 0.0 0.0"/>
-    <parent link="Index_Proximal"/>
-    <child link="Index_Middle"/>
-    <dynamics damping="0.1"/>
-    <limit effort="0.5" lower="0" upper="1.57079632679" velocity="1.0"/>
+        <origin xyz="6.2440782901e-05 0 -0.025875292969" rpy="0 0 0"/>
+        <axis xyz="-1.0 0.0 0.0"/>
+        <parent link="Index_Proximal"/>
+        <child link="Index_Middle"/>
+        <mimic joint="Index_Proximal--palmL:1"
+                multiplier="0.9"
+                offset="0.0"/>
+        <dynamics damping="0.02" friction="0.0"/>
+        <limit effort="2.5" lower="0" upper="1.57079632679" velocity="5.0"/>
     </joint>
     <!-- Index Distal -->
@@ -90,10 +93,13 @@
     <!--Joint: Index_Middle -> Index_Distal -->
     <joint name="Index_Distal--Index_Middle" type="revolute">
-    <origin xyz="6.2578385226e-05 -2.1183475668e-07 -0.0258743408417" rpy="0 0 0"/>
-    <axis xyz="-1.0 0.0 0.0"/>
-    <parent link="Index_Middle"/>
-    <child link="Index_Distal"/>
-    <dynamics damping="0.1"/>
-    <limit effort="0.5" lower="0" upper="1.57079632679" velocity="1.0"/>
+        <origin xyz="6.2578385226e-05 -2.1183475668e-07 -0.0258743408417" rpy="0 0 0"/>
+        <axis xyz="-1.0 0.0 0.0"/>
+        <parent link="Index_Middle"/>
+        <child link="Index_Distal"/>
+        <mimic joint="Index_Middle--Index_Proximal"
+                multiplier="0.9"
+                offset="0.0"/>
+        <dynamics damping="0.02" friction="0.0"/>
+        <limit effort="2.5" lower="0" upper="1.57079632679" velocity="5.0"/>
     </joint>
 </robot>

File: v2_rh8d_ws/src/rh8d_description/urdf/rh8dL_main.urdf (robot description, URDF)
Before this commit: robot RH8DL, 21 links, 20 joints
Links:
- removed link base_link
- added link world
Joints:
- removed joint base:1--base_link
- added joint base:1--world: type fixed, parent world, child base:1, origin xyz=0.58 -0.13 1.045 rpy=-1.57079632679 0 0
- joint Index_Distal--Index_Middle: limit lower=0 upper=1.57079632679 effort=0.5 velocity=1.0 -> lower=0 upper=1.57079632679 effort=2.5 velocity=5.0; mimic (none) -> joint=Index_Middle--Index_Proximal multiplier=0.9 offset=0.0
- joint Index_Middle--Index_Proximal: limit lower=0 upper=1.57079632679 effort=0.5 velocity=1.0 -> lower=0 upper=1.57079632679 effort=2.5 velocity=5.0; mimic (none) -> joint=Index_Proximal--palmL:1 multiplier=0.9 offset=0.0
- joint Index_Proximal--palmL:1: limit lower=0 upper=1.57079632679 effort=0.5 velocity=1.0 -> lower=0 upper=1.57079632679 effort=2.5 velocity=5.0
- joint Middle_Distal--Middle_Middle: limit lower=0 upper=1.57079632679 effort=0.5 velocity=1.0 -> lower=0 upper=1.57079632679 effort=2.5 velocity=5.0; mimic (none) -> joint=Middle_Middle--Middle_Proximal multiplier=0.9 offset=0.0
- joint Middle_Middle--Middle_Proximal: limit lower=0 upper=1.57079632679 effort=0.5 velocity=1.0 -> lower=0 upper=1.57079632679 effort=2.5 velocity=5.0; mimic (none) -> joint=Middle_Proximal--palmL:1 multiplier=0.9 offset=0.0
- joint Middle_Proximal--palmL:1: limit lower=0 upper=1.57079632679 effort=0.5 velocity=1.0 -> lower=0 upper=1.57079632679 effort=2.5 velocity=5.0
- joint Ring_Distal--Ring_Middle: limit lower=0 upper=1.57079632679 effort=0.5 velocity=1.0 -> lower=0 upper=1.57079632679 effort=0.5 velocity=10.0; mimic (none) -> joint=Ring_Middle--Ring_Proximal multiplier=0.9 offset=0.0
- joint Ring_Middle--Ring_Proximal: limit lower=0 upper=1.57079632679 effort=0.5 velocity=1.0 -> lower=0 upper=1.57079632679 effort=0.5 velocity=10.0; mimic (none) -> joint=Ring_Proximal--palmL:1 multiplier=0.9 offset=0.0
- joint Ring_Proximal--palmL:1: limit lower=0 upper=1.57079632679 effort=0.5 velocity=1.0 -> lower=0 upper=1.57079632679 effort=0.5 velocity=10.0
- joint Small_Distal--Small_Middle: limit lower=0 upper=1.57079632679 effort=0.5 velocity=1.0 -> lower=0 upper=1.57079632679 effort=0.5 velocity=10.0; mimic (none) -> joint=Small_Middle--Small_Proximal multiplier=0.9 offset=0.0
- joint Small_Middle--Small_Proximal: limit lower=0 upper=1.57079632679 effort=0.5 velocity=1.0 -> lower=0 upper=1.57079632679 effort=0.5 velocity=10.0; mimic (none) -> joint=Small_Proximal--palmL:1 multiplier=0.9 offset=0.0
- joint Small_Proximal--palmL:1: limit lower=0 upper=1.57079632679 effort=0.5 velocity=1.0 -> lower=0 upper=1.57079632679 effort=0.5 velocity=10.0; mimic (none) -> joint=Ring_Proximal--palmL:1 multiplier=1.0 offset=0.0
- joint Thumb_Distal--Thumb_Proximal: limit lower=-1.57079632679 upper=1.57079632679 effort=0.5 velocity=1.0 -> lower=0.0 upper=1.57079632679 effort=2.5 velocity=5.0; mimic (none) -> joint=Thumb_Proximal--Thumb_Methacarpal multiplier=0.9 offset=0.0
- joint Thumb_Methacarpal--Thumb_axis: limit lower=-1.57079632679 upper=1.57079632679 effort=0.5 velocity=1.0 -> lower=0.0 upper=1.57079632679 effort=2.5 velocity=5.0
- joint Thumb_Proximal--Thumb_Methacarpal: limit lower=-1.57079632679 upper=1.57079632679 effort=0.5 velocity=1.0 -> lower=0.0 upper=1.57079632679 effort=2.5 velocity=5.0; mimic (none) -> joint=Thumb_Methacarpal--Thumb_axis multiplier=0.9 offset=0.0
- joint Thumb_axis--palmL:1: limit lower=0 upper=1.57079632679 effort=0.5 velocity=1.0 -> lower=-0.001 upper=1.57079632679 effort=2.5 velocity=5.0
- joint forearm:1--base:1: limit lower=-1.57079632679 upper=1.57079632679 effort=0.5 velocity=1.0 -> lower=-1.57079632679 upper=1.57079632679 effort=2.5 velocity=5.0
- joint palmL:1--palm_axis:1: limit lower=-0.785398163395 upper=0.785398163395 effort=0.5 velocity=1.0 -> lower=-0.785398163395 upper=0.785398163395 effort=2.5 velocity=5.0
- joint palm_axis:1--forearm:1: limit lower=-1.57079632679 upper=1.57079632679 effort=0.5 velocity=1.0 -> lower=-1.57079632679 upper=1.57079632679 effort=2.5 velocity=5.0

File: v2_rh8d_ws/src/rh8d_description/urdf/rh8dL_middle.xacro (robot description, xacro)
@@ -26,10 +26,10 @@
     <!-- Joint: palmL:1 -> Middle_Proximal -->
     <joint name="Middle_Proximal--palmL:1" type="revolute">
-    <origin xyz="-0.0095654 -0.082818 0.00164059" rpy="-1.74598210711 -0.0859373918966 0.0151910468121"/>
-    <axis xyz="-1.0 0.0 0.0"/>
-    <parent link="palmL:1"/>
-    <child link="Middle_Proximal"/>
-    <dynamics damping="0.1"/>
-    <limit effort="0.5" lower="0" upper="1.57079632679" velocity="1.0"/>
+        <origin xyz="-0.0095654 -0.082818 0.00164059" rpy="-1.74598210711 -0.0859373918966 0.0151910468121"/>
+        <axis xyz="-1.0 0.0 0.0"/>
+        <parent link="palmL:1"/>
+        <child link="Middle_Proximal"/>
+        <dynamics damping="0.05" friction="0.005"/>
+        <limit effort="2.5" lower="0" upper="1.57079632679" velocity="5.0"/>
     </joint>
     <!-- Middle Middle -->
@@ -58,10 +58,13 @@
     <!-- Joint: Middle_Proximal -> Middle_Middle -->
     <joint name="Middle_Middle--Middle_Proximal" type="revolute">
-    <origin xyz="6.25377180185e-05 0 -0.0258750444163" rpy="0 0 0"/>
-    <axis xyz="-1.0 0.0 0.0"/>
-    <parent link="Middle_Proximal"/>
-    <child link="Middle_Middle"/>
-    <dynamics damping="0.1"/>
-    <limit effort="0.5" lower="0" upper="1.57079632679" velocity="1.0"/>
+        <origin xyz="6.25377180185e-05 0 -0.0258750444163" rpy="0 0 0"/>
+        <axis xyz="-1.0 0.0 0.0"/>
+        <parent link="Middle_Proximal"/>
+        <child link="Middle_Middle"/>
+        <mimic joint="Middle_Proximal--palmL:1"
+                multiplier="0.9"
+                offset="0.0"/>
+        <dynamics damping="0.02" friction="0.0"/>
+        <limit effort="2.5" lower="0" upper="1.57079632679" velocity="5.0"/>
     </joint>
     <!-- Middle Distal -->
@@ -90,10 +93,13 @@
     <!-- Joint: Middle_Middle -> Middle_Distal -->
     <joint name="Middle_Distal--Middle_Middle" type="revolute">
-    <origin xyz="6.24372402321e-05 0 -0.0258750426798" rpy="0 0 0"/>
-    <axis xyz="-1.0 0.0 0.0"/>
-    <parent link="Middle_Middle"/>
-    <child link="Middle_Distal"/>
-    <dynamics damping="0.1"/>
-    <limit effort="0.5" lower="0" upper="1.57079632679" velocity="1.0"/>
+        <origin xyz="6.24372402321e-05 0 -0.0258750426798" rpy="0 0 0"/>
+        <axis xyz="-1.0 0.0 0.0"/>
+        <parent link="Middle_Middle"/>
+        <child link="Middle_Distal"/>
+        <mimic joint="Middle_Middle--Middle_Proximal"
+            multiplier="0.9"
+            offset="0.0"/>
+        <dynamics damping="0.02" friction="0.0"/>
+        <limit effort="2.5" lower="0" upper="1.57079632679" velocity="5.0"/>
     </joint>
 </robot>
