Commit message: Under-actuated RH8D Gazebo simulation

File: v2_rh8d_ws/src/rh8d_description/urdf/rh8dL_palm.xacro (robot description, xacro)
@@ -26,11 +26,10 @@
     <!-- Joint: forearm:1 -> palm_axis:1 -->
     <joint name="palm_axis:1--forearm:1" type="revolute">
-    <origin xyz="0 -0.165 -0.01275" rpy="0 0 0"/>
-    <axis xyz="0.0 0.0 -1.0"/>
-    <parent link="forearm:1"/>
-    <child link="palm_axis:1"/>
-    <dynamics damping="0.1"/>
-    <!-- <limit effort="0.5" lower="-0.785398163395" upper="0.785398163395" velocity="1.0"/> -->
-    <limit effort="0.5" lower="-1.57079632679" upper="1.57079632679" velocity="1.0"/>
+        <origin xyz="0 -0.165 -0.01275" rpy="0 0 0"/>
+        <axis xyz="0.0 0.0 -1.0"/>
+        <parent link="forearm:1"/>
+        <child link="palm_axis:1"/>
+        <dynamics damping="0.05" friction="0.005"/>
+        <limit effort="2.5" lower="-1.57079632679" upper="1.57079632679" velocity="5.0"/>
     </joint>
     <!-- Palm L:1 -->
@@ -59,10 +58,10 @@
     <!-- Joint: palm_axis:1 -> palmL:1 -->
     <joint name="palmL:1--palm_axis:1" type="revolute">
-    <origin xyz="-0.0265 0 0.0125" rpy="3.14159265359 0 3.14159265359"/>
-    <axis xyz="-1.0 0.0 0.0"/>
-    <parent link="palm_axis:1"/>
-    <child link="palmL:1"/>
-    <dynamics damping="0.1"/>
-    <limit effort="0.5" lower="-0.785398163395" upper="0.785398163395" velocity="1.0"/>
+        <origin xyz="-0.0265 0 0.0125" rpy="3.14159265359 0 3.14159265359"/>
+        <axis xyz="-1.0 0.0 0.0"/>
+        <parent link="palm_axis:1"/>
+        <child link="palmL:1"/>
+        <dynamics damping="0.05" friction="0.005"/>
+        <limit effort="2.5" lower="-0.785398163395" upper="0.785398163395" velocity="5.0"/>
     </joint>
 </robot>

File: v2_rh8d_ws/src/rh8d_description/urdf/rh8dL_ring.xacro (robot description, xacro)
@@ -26,10 +26,10 @@
     <!-- Joint: palmL:1 -> Ring_Proximal -->
     <joint name="Ring_Proximal--palmL:1" type="revolute">
-    <origin xyz="-0.03444198 -0.082386 0.00076556" rpy="-1.75269165877 0.0686359653419 -0.101002048759"/>
-    <axis xyz="-1.0 0.0 0.0"/>
-    <parent link="palmL:1"/>
-    <child link="Ring_Proximal"/>
-    <dynamics damping="0.1"/>
-    <limit effort="0.5" lower="0" upper="1.57079632679" velocity="1.0"/>
+        <origin xyz="-0.03444198 -0.082386 0.00076556" rpy="-1.75269165877 0.0686359653419 -0.101002048759"/>
+        <axis xyz="-1.0 0.0 0.0"/>
+        <parent link="palmL:1"/>
+        <child link="Ring_Proximal"/>
+        <dynamics damping="0.05" friction="0.005"/>
+        <limit effort="0.5" lower="0" upper="1.57079632679" velocity="10.0"/>
     </joint>
     <!-- Ring Middle -->
@@ -62,6 +62,9 @@
     <parent link="Ring_Proximal"/>
     <child link="Ring_Middle"/>
-    <dynamics damping="0.1"/>
-    <limit effort="0.5" lower="0" upper="1.57079632679" velocity="1.0"/>
+    <mimic joint="Ring_Proximal--palmL:1"
+                multiplier="0.9"
+                offset="0.0"/>
+    <dynamics damping="0.02" friction="0.0"/>
+    <limit effort="0.5" lower="0" upper="1.57079632679" velocity="10.0"/>
     </joint>
     <!-- Ring Distal -->
@@ -90,10 +93,13 @@
     <!-- Joint: Ring_Middle -> Ring_Distal -->
     <joint name="Ring_Distal--Ring_Middle" type="revolute">
-    <origin xyz="6.25316406279e-05 1.7655252639e-07 -0.0258758931888" rpy="0 0 0"/>
-    <axis xyz="-1.0 0.0 0.0"/>
-    <parent link="Ring_Middle"/>
-    <child link="Ring_Distal"/>
-    <dynamics damping="0.1"/>
-    <limit effort="0.5" lower="0" upper="1.57079632679" velocity="1.0"/>
+        <origin xyz="6.25316406279e-05 1.7655252639e-07 -0.0258758931888" rpy="0 0 0"/>
+        <axis xyz="-1.0 0.0 0.0"/>
+        <parent link="Ring_Middle"/>
+        <child link="Ring_Distal"/>
+        <mimic joint="Ring_Middle--Ring_Proximal"
+                    multiplier="0.9"
+                    offset="0.0"/>
+        <dynamics damping="0.02" friction="0.0"/>
+        <limit effort="0.5" lower="0" upper="1.57079632679" velocity="10.0"/>
     </joint>
 </robot>

File: v2_rh8d_ws/src/rh8d_description/urdf/rh8dL_small.xacro (robot description, xacro)
@@ -26,10 +26,13 @@
     <!-- Joint: palmL:1 -> Small_Proximal -->
     <joint name="Small_Proximal--palmL:1" type="revolute">
-    <origin xyz="-0.0591609 -0.07417 0.00246184" rpy="-1.77486172903 0.138702392285 -0.20406540224"/>
-    <axis xyz="-1.0 0.0 0.0"/>
-    <parent link="palmL:1"/>
-    <child link="Small_Proximal"/>
-    <dynamics damping="0.1"/>
-    <limit effort="0.5" lower="0" upper="1.57079632679" velocity="1.0"/>
+        <origin xyz="-0.0591609 -0.07417 0.00246184" rpy="-1.77486172903 0.138702392285 -0.20406540224"/>
+        <axis xyz="-1.0 0.0 0.0"/>
+        <parent link="palmL:1"/>
+        <child link="Small_Proximal"/>
+        <mimic joint="Ring_Proximal--palmL:1"
+                    multiplier="1.0"
+                    offset="0.0"/>
+        <dynamics damping="0.002" friction="0.0"/>
+        <limit effort="0.5" lower="0" upper="1.57079632679" velocity="10.0"/>
     </joint>
     <!-- Small Middle -->
@@ -58,10 +61,13 @@
     <!-- Joint: Small_Proximal -> Small_Middle -->
     <joint name="Small_Middle--Small_Proximal" type="revolute">
-    <origin xyz="6.25112164948e-05 0 -0.0258751651529" rpy="0 0 0"/>
-    <axis xyz="-1.0 0.0 0.0"/>
-    <parent link="Small_Proximal"/>
-    <child link="Small_Middle"/>
-    <dynamics damping="0.1"/>
-    <limit effort="0.5" lower="0" upper="1.57079632679" velocity="1.0"/>
+        <origin xyz="6.25112164948e-05 0 -0.0258751651529" rpy="0 0 0"/>
+        <axis xyz="-1.0 0.0 0.0"/>
+        <parent link="Small_Proximal"/>
+        <child link="Small_Middle"/>
+        <mimic joint="Small_Proximal--palmL:1"
+                    multiplier="0.9"
+                    offset="0.0"/>
+        <dynamics damping="0.002" friction="0.0"/>
+        <limit effort="0.5" lower="0" upper="1.57079632679" velocity="10.0"/>
     </joint>
     <!-- Small Distal -->
@@ -94,6 +100,9 @@
     <parent link="Small_Middle"/>
     <child link="Small_Distal"/>
-    <dynamics damping="0.1"/>
-    <limit effort="0.5" lower="0" upper="1.57079632679" velocity="1.0"/>
+    <mimic joint="Small_Middle--Small_Proximal"
+                multiplier="0.9"
+                offset="0.0"/>
+    <dynamics damping="0.002" friction="0.0"/>
+    <limit effort="0.5" lower="0" upper="1.57079632679" velocity="10.0"/>
     </joint>
 </robot>

File: v2_rh8d_ws/src/rh8d_description/urdf/rh8dL_thumb.xacro (robot description, xacro)
@@ -26,10 +26,10 @@
     <!-- Joint: palmL:1 -> Thumb_axis -->
     <joint name="Thumb_axis--palmL:1" type="revolute">
-    <origin xyz="-0.0078751 -0.035115 0.00101669" rpy="-1.57079652646 -1.26729978315 -1.81210600928"/>
-    <axis xyz="0.0 0.866025655797 -0.5000003546"/>
-    <parent link="palmL:1"/>
-    <child link="Thumb_axis"/>
-    <dynamics damping="0.1"/>
-    <limit effort="0.5" lower="0" upper="1.57079632679" velocity="1.0"/>
+        <origin xyz="-0.0078751 -0.035115 0.00101669" rpy="-1.57079652646 -1.26729978315 -1.81210600928"/>
+        <axis xyz="0.0 0.866025655797 -0.5000003546"/>
+        <parent link="palmL:1"/>
+        <child link="Thumb_axis"/>
+        <dynamics damping="0.04" friction="0.005"/>
+        <limit effort="2.5" lower="-0.001" upper="1.57079632679" velocity="5.0"/>
     </joint>
     <!-- Thumb Methacarpal -->
@@ -58,10 +58,10 @@
     <!-- Joint: Thumb_axis -> Thumb_Methacarpal -->
     <joint name="Thumb_Methacarpal--Thumb_axis" type="revolute">
-    <origin xyz="-0.00512499670326 -0.0143547805534 0.0211783500758" rpy="3.14159265359 0 0"/>
-    <axis xyz="-1.0 0.0 0.0"/>
-    <parent link="Thumb_axis"/>
-    <child link="Thumb_Methacarpal"/>
-    <dynamics damping="0.1"/>
-    <limit effort="0.5" lower="-1.57079632679" upper="1.57079632679" velocity="1.0"/>
+        <origin xyz="-0.00512499670326 -0.0143547805534 0.0211783500758" rpy="3.14159265359 0 0"/>
+        <axis xyz="-1.0 0.0 0.0"/>
+        <parent link="Thumb_axis"/>
+        <child link="Thumb_Methacarpal"/>
+        <dynamics damping="0.04" friction="0.005"/>
+        <limit effort="2.5" lower="-0.001" upper="1.57079632679" velocity="5.0"/>
     </joint>
     <!-- Thumb Proximal -->
@@ -90,10 +90,13 @@
     <!-- Joint: Thumb_Methacarpal -> Thumb_Proximal -->
     <joint name="Thumb_Proximal--Thumb_Methacarpal" type="revolute">
-    <origin xyz="-0.000562285554381 -6.82918828571e-07 -0.021586139018" rpy="0 0 0"/>
-    <axis xyz="-1.0 0.0 0.0"/>
-    <parent link="Thumb_Methacarpal"/>
-    <child link="Thumb_Proximal"/>
-    <dynamics damping="0.1"/>
-    <limit effort="0.5" lower="-1.57079632679" upper="1.57079632679" velocity="1.0"/>
+        <origin xyz="-0.000562285554381 -6.82918828571e-07 -0.021586139018" rpy="0 0 0"/>
+        <axis xyz="-1.0 0.0 0.0"/>
+        <parent link="Thumb_Methacarpal"/>
+        <child link="Thumb_Proximal"/>
+        <mimic joint="Thumb_Methacarpal--Thumb_axis"
+                multiplier="0.9"
+                offset="0.0"/>
+        <dynamics damping="0.02" friction="0.0"/>
+        <limit effort="2.5" lower="-0.001" upper="1.57079632679" velocity="5.0"/>
     </joint>
     <!-- Thumb Distal -->
@@ -122,10 +125,13 @@
     <!-- Joint: Thumb_Proximal -> Thumb_Distal -->
     <joint name="Thumb_Distal--Thumb_Proximal" type="revolute">
-    <origin xyz="-6.26114843445e-05 3.61581448449e-07 -0.0215859828359" rpy="0 0 0"/>
-    <axis xyz="-1.0 0.0 0.0"/>
-    <parent link="Thumb_Proximal"/>
-    <child link="Thumb_Distal"/>
-    <dynamics damping="0.1"/>
-    <limit effort="0.5" lower="-1.57079632679" upper="1.57079632679" velocity="1.0"/>
+        <origin xyz="-6.26114843445e-05 3.61581448449e-07 -0.0215859828359" rpy="0 0 0"/>
+        <axis xyz="-1.0 0.0 0.0"/>
+        <parent link="Thumb_Proximal"/>
+        <child link="Thumb_Distal"/>
+        <mimic joint="Thumb_Proximal--Thumb_Methacarpal"
+                multiplier="0.9"
+                offset="0.0"/>
+        <dynamics damping="0.02" friction="0.0"/>
+        <limit effort="2.5" lower="-0.001" upper="1.57079632679" velocity="5.0"/>
     </joint>
 </robot>
